File: Version2.1/PiStorm2k_v2.1.kicad_pcb (KiCad board)
At the start: 4 copper layers, 135.2 x 96.5 mm, 57 parts, among them J1 CONN_171826-4_TYCO_TYC, P78 TestPoint_Pad_1.0x1.0mm, P81 TestPoint_Pad_1.0x1.0mm, P82 TestPoint_Pad_1.0x1.0mm, P83 TestPoint_Pad_1.0x1.0mm, U1 SN74LVC16374DGGR, U10 VREG_LM1117IMPX-3.3, U11 VREG_LM1117IMPX-3.3, U2 SN74LVC16374DGGR, U3 SN74CBTD3384PWR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

Commit message: Add files via upload
Parts:
- removed PI: Header 20X2, Copy of ps32-lite_45_padshapes.PcbLib:CONN-SMD_FH-00369
